File: PCB Files/Cerebro 5.8/cerebro5.8.sch (EAGLE design)
At the start: 49 parts, among them T1 FJX3904TF, T2 FJX3904TF, U2 915MHz, U3 Fuel Guage

Commit message: Updated to latest PCB files
Parts:
- removed S3: (no value), Cerebro-library:SWITCH-SPDTSMD2
- removed U$2, U$3: ANTENNA, Cerebro-library:ANTENNA
- added INDICATOR_LED2: GRN, led:LEDCHIP-LED0603
- added R10: 4.7k, Cerebro-library:RESISTOR0603-RES
- added RESET1: SWITCH-MOMENTARY-NO, Cerebro-library:SWITCH-MOMENTARY-NO
- added S1: (no value), Cerebro-library:SWITCH-SPDTREINFORCED_SMD
- CN1: device Cerebro-library:JST-SRJS-1MM -> Cerebro-library:JST_2PINMICRO
- DAC1, DAC2: value DAC_LTC2630 -> DAC
- INDICATOR_LED1: value AMBER -> YLW
- R12, R13: value 22 -> 27
- R18, R19: value 10k -> 20k
- R20: value 20k -> 4.7k
Connections:
- removed net N$32: U$4.PD6(ADC9)
- new net N$20: INDICATOR_LED2.C, R10.1
- new net N$21: RESET1.1, U$4.PD7(ADC10)
- net BAT_IN: now also S1.P; no longer S3.P
- net GND: now also R10.2, RESET1.2, S1.O; no longer S3.S, U$3.1
- net N$29: now also INDICATOR_LED2.A, U$4.PD6(ADC9); no longer U$4.PD7(ADC10)
- net N$4: now also S1.S; no longer S3.O
- net RESET: no longer U$2.1
